File: Hardware/Electric+Scheme.sch (EAGLE design)
At the start: 103 parts, among them IC1 BD5229G-TR, IC4 XC6220A331MR-G, J1 FH34SRJ-24S-0.5SH_99_, J2 SAMACSYS_PARTS_USB4110-GF-A, J3 QWIIC_RIGHT_ANGLE, J4 112A-TAAR-R03_ATTEND, Q1 20V/4.2A/52mΩ/1.4W, Q2 20V/4.2A/52mΩ/1.4W, Q3 SI1308EDL-T1-GE3, U1 W25Q512JVEIQ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

Commit message: Add files via upload
Parts:
- CHG_LED: value (none) -> RED
- SJ1: value (none) -> SOLDERJUMPER
Connections:
- removed net N$7: J3.4
- new net N$15: EPD_C12.2, J1.24
- net GND: now also J1.MP1, J1.MP2
- net N$4: now also J2.B5, R2-USB.1; no longer J3.3
- net PREVGL: no longer EPD_C12.2, J1.24, J1.MP1, J1.MP2
- net SCL: now also J3.4
- net SDA: now also J3.3
Changed lines of the file:
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@@
 <part name="SUPPLY2" library="Power_Symbols" library_urn="urn:adsk.eagle:library:16502351" deviceset="GND-BAR" device="" value="GND"/>
 <part name="SUPPLY3" library="Power_Symbols" library_urn="urn:adsk.eagle:library:16502351" deviceset="GND-BAR" device="" value="GND"/>
-<part name="FRAME1" library="DeskAssistant v19 v1" library_urn="urn:adsk.wipprod:fs.file:vf.H3hVZ9NQS92JNyqNQFLgCQ" deviceset="ESP32_WROVER_FRAMES_A3L-LOC" device=""/>
+<part name="FRAME1" library="DeskAssistant v19 v1" library_urn="urn:adsk.wipprod:fs.file:vf.H3hVZ9NQS92JNyqNQFLgCQ" deviceset="ESP32_WROVER_FRAMES_A3L-LOC" device="" value="OpenBook Schematic"/>
 <part name="U2" library="DeskAssistant v19 v1" library_urn="urn:adsk.wipprod:fs.file:vf.H3hVZ9NQS92JNyqNQFLgCQ" deviceset="ESP32-C6-WROOM-1-N8" device=""/>
 <part name="SUPPLY4" library="Power_Symbols" library_urn="urn:adsk.eagle:library:16502351" deviceset="VCC-CIRCLE" device="" value="3V3"/>
@@
 <part name="GND9" library="DeskAssistant v19 v1" library_urn="urn:adsk.wipprod:fs.file:vf.H3hVZ9NQS92JNyqNQFLgCQ" deviceset="GND" device=""/>
 <part name="GND10" library="DeskAssistant v19 v1" library_urn="urn:adsk.wipprod:fs.file:vf.H3hVZ9NQS92JNyqNQFLgCQ" deviceset="GND" device=""/>
-<part uuid="2882400012" name="SJ1" library="DeskAssistant v19 v1" library_urn="urn:adsk.wipprod:fs.file:vf.H3hVZ9NQS92JNyqNQFLgCQ" deviceset="SJ" device=""/>
+<part uuid="2882400012" name="SJ1" library="DeskAssistant v19 v1" library_urn="urn:adsk.wipprod:fs.file:vf.H3hVZ9NQS92JNyqNQFLgCQ" deviceset="SJ" device="" value="SOLDERJUMPER"/>
 <part name="GND11" library="DeskAssistant v19 v1" library_urn="urn:adsk.wipprod:fs.file:vf.H3hVZ9NQS92JNyqNQFLgCQ" deviceset="GND" device=""/>
 <part name="R2" library="DeskAssistant v19 v1" library_urn="urn:adsk.wipprod:fs.file:vf.H3hVZ9NQS92JNyqNQFLgCQ" deviceset="ESP32_WROVER_EAGLE-LTSPICE_R" device="" value="2.2"/>
@@
 <part uuid="2882400035" name="MCP73831" library="DeskAssistant v19 v1" library_urn="urn:adsk.wipprod:fs.file:vf.H3hVZ9NQS92JNyqNQFLgCQ" deviceset="ESP32_WROVER_SPARKFUN-IC-POWER_MCP73831" device=""/>
 <part name="R1_BAT" library="DeskAssistant v19 v1" library_urn="urn:adsk.wipprod:fs.file:vf.H3hVZ9NQS92JNyqNQFLgCQ" deviceset="ESP32_WROVER_EAGLE-LTSPICE_R" device="" value="200"/>
-<part uuid="2882400053" name="CHG_LED" library="DeskAssistant v19 v1" library_urn="urn:adsk.wipprod:fs.file:vf.H3hVZ9NQS92JNyqNQFLgCQ" deviceset="ADAFRUIT_LED" device="CHIP-LED0603"/>
+<part uuid="2882400053" name="CHG_LED" library="DeskAssistant v19 v1" library_urn="urn:adsk.wipprod:fs.file:vf.H3hVZ9NQS92JNyqNQFLgCQ" deviceset="ADAFRUIT_LED" device="CHIP-LED0603" value="RED"/>
 <part name="C1_BAT" library="DeskAssistant v19 v1" library_urn="urn:adsk.wipprod:fs.file:vf.H3hVZ9NQS92JNyqNQFLgCQ" deviceset="EAGLE-LTSPICE_C" device="" value="4.7uF"/>
 <part name="GND16" library="DeskAssistant v19 v1" library_urn="urn:adsk.wipprod:fs.file:vf.H3hVZ9NQS92JNyqNQFLgCQ" deviceset="GND" device=""/>
@@
 <instance part="SJ1" gate="1" x="213.36" y="-22.86" smashed="yes">
 <attribute name="NAME" x="210.82" y="-20.32" size="1.778" layer="95"/>
-<attribute name="VALUE" x="210.82" y="-26.67" size="1.778" layer="96"/>
 </instance>
 <instance part="GND11" gate="1" x="200.66" y="-27.94" smashed="yes">
@@
 <instance part="CHG_LED" gate="G$1" x="388.62" y="-35.56" smashed="yes">
 <attribute name="NAME" x="392.176" y="-40.132" size="1.778" layer="95" rot="R90"/>
-<attribute name="VALUE" x="394.335" y="-40.132" size="1.778" layer="96" rot="R90"/>
 </instance>
 <instance part="C1_BAT" gate="G$1" x="370.84" y="-35.56" smashed="yes">
@@
 <attribute name="VALUE" x="266.7" y="-133.35" size="1.778" layer="96" rot="MR90" align="center-left"/>
 </instance>
-<instance part="SUPPLY21" gate="G$1" x="274.32" y="-76.2" smashed="yes">
-<attribute name="VALUE" x="274.32" y="-78.105" size="1.778" layer="96" align="center"/>
+<instance part="SUPPLY21" gate="G$1" x="276.86" y="-81.28" smashed="yes">
+<attribute name="VALUE" x="276.86" y="-83.185" size="1.778" layer="96" align="center"/>
 </instance>
 <instance part="EPD_C2" gate="G$1" x="226.06" y="-121.92" smashed="yes" rot="R90">
@@
 <pinref part="CHANGE_BUTTON" gate="G$1" pin="2"/>
 </segment>
+<segment>
+<pinref part="J1" gate="G$1" pin="MP2"/>
+<wire x1="269.24" y1="-73.66" x2="276.86" y2="-73.66" width="0.1524" layer="91"/>
+<wire x1="276.86" y1="-73.66" x2="276.86" y2="-76.2" width="0.1524" layer="91"/>
+<pinref part="SUPPLY21" gate="G$1" pin="GND"/>
+<pinref part="J1" gate="G$1" pin="MP1"/>
+<wire x1="276.86" y1="-76.2" x2="276.86" y2="-78.74" width="0.1524" layer="91"/>
+<wire x1="269.24" y1="-76.2" x2="276.86" y2="-76.2" width="0.1524" layer="91"/>
+<junction x="276.86" y="-76.2"/>
+</segment>
 </net>
 <net name="MOSI" class="0">
@@
 <pinref part="R2-PINH" gate="G$1" pin="1"/>
 </segment>
+<segment>
+<pinref part="J3" gate="J1" pin="4"/>
+<wire x1="381" y1="-190.5" x2="378.46" y2="-190.5" width="0.1524" layer="91"/>
+<label x="378.46" y="-190.5" size="1.016" layer="95" rot="R180" xref="yes"/>
+</segment>
 </net>
 <net name="SDA" class="0">
@@
 <label x="388.62" y="-106.68" size="1.016" layer="95" rot="R270" xref="yes"/>
 <pinref part="R1-PINH" gate="G$1" pin="1"/>
+</segment>
+<segment>
+<pinref part="J3" gate="J1" pin="3"/>
+<wire x1="381" y1="-187.96" x2="378.46" y2="-187.96" width="0.1524" layer="91"/>
+<label x="378.46" y="-187.96" size="1.016" layer="95" rot="R180" xref="yes"/>
 </segment>
 </net>
@@
 </segment>
 <segment>
-<pinref part="J1" gate="G$1" pin="24"/>
-<wire x1="269.24" y1="-73.66" x2="274.32" y2="-73.66" width="0.1524" layer="91"/>
-<wire x1="274.32" y1="-73.66" x2="274.32" y2="-76.2" width="0.1524" layer="91"/>
-<wire x1="274.32" y1="-76.2" x2="269.24" y2="-76.2" width="0.1524" layer="91"/>
 <pinref part="J1" gate="G$1" pin="23"/>
-<pinref part="SUPPLY21" gate="G$1" pin="GND"/>
-<pinref part="J1" gate="G$1" pin="MP1"/>
-<pinref part="J1" gate="G$1" pin="MP2"/>
-<wire x1="243.84" y1="-73.66" x2="236.22" y2="-73.66" width="0.1524" layer="91"/>
 <wire x1="243.84" y1="-76.2" x2="241.3" y2="-76.2" width="0.1524" layer="91"/>
-<junction x="274.32" y="-73.66"/>
-<wire x1="241.3" y1="-76.2" x2="220.98" y2="-76.2" width="0.1524" layer="91"/>
-<junction x="241.3" y="-76.2"/>
-<wire x1="241.3" y1="-76.2" x2="241.3" y2="-68.58" width="0.1524" layer="91"/>
 <label x="241.3" y="-68.58" size="1.016" layer="95" rot="R90" xref="yes"/>
 <pinref part="EPD_C11" gate="G$1" pin="2"/>
-<pinref part="EPD_C12" gate="G$1" pin="2"/>
+<wire x1="241.3" y1="-76.2" x2="220.98" y2="-76.2" width="0.1524" layer="91"/>
+<wire x1="241.3" y1="-68.58" x2="241.3" y2="-76.2" width="0.1524" layer="91"/>
+<junction x="241.3" y="-76.2"/>
 </segment>
 </net>
@@
 <segment>
 <pinref part="J1" gate="G$1" pin="21"/>
-<wire x1="243.84" y1="-81.28" x2="236.22" y2="-81.28" width="0.1524" layer="91"/>
-<wire x1="236.22" y1="-81.28" x2="220.98" y2="-81.28" width="0.1524" layer="91"/>
-<junction x="236.22" y="-81.28"/>
-<wire x1="236.22" y1="-81.28" x2="236.22" y2="-71.12" width="0.1524" layer="91"/>
-<label x="236.22" y="-71.12" size="1.016" layer="95" rot="R90" xref="yes"/>
+<wire x1="243.84" y1="-81.28" x2="238.76" y2="-81.28" width="0.1524" layer="91"/>
+<label x="238.76" y="-71.12" size="1.016" layer="95" rot="R90" xref="yes"/>
 <pinref part="EPD_C9" gate="G$1" pin="2"/>
+<wire x1="238.76" y1="-81.28" x2="220.98" y2="-81.28" width="0.1524" layer="91"/>
+<wire x1="238.76" y1="-71.12" x2="238.76" y2="-81.28" width="0.1524" layer="91"/>
+<junction x="238.76" y="-81.28"/>
 </segment>
 </net>
 <net name="EPD_3V3" class="1">
 <segment>
+<wire x1="243.84" y1="-33.02" x2="243.84" y2="-30.48" width="0.1524" layer="91"/>
+<label x="243.84" y="-25.4" size="1.016" layer="95" rot="R90" xref="yes"/>
+<pinref part="C7" gate="G$1" pin="1"/>
+<pinref part="L1" gate="A" pin="2"/>
+<wire x1="243.84" y1="-30.48" x2="243.84" y2="-25.4" width="0.1524" layer="91"/>
 <wire x1="246.38" y1="-30.48" x2="243.84" y2="-30.48" width="0.1524" layer="91"/>
-<wire x1="243.84" y1="-30.48" x2="243.84" y2="-25.4" width="0.1524" layer="91"/>
-<wire x1="243.84" y1="-30.48" x2="243.84" y2="-33.02" width="0.1524" layer="91"/>
-<label x="243.84" y="-25.4" size="1.016" layer="95" rot="R90" xref="yes"/>
-<pinref part="L1" gate="A" pin="2"/>
-<pinref part="C7" gate="G$1" pin="1"/>
+<junction x="243.84" y="-30.48"/>
 </segment>
 <segment>
@@
 <pinref part="R10" gate="G$1" pin="1"/>
 <pinref part="D8" gate="G$1" pin="2"/>
-</segment>
-</net>
-<net name="N$4" class="0">
-<segment>
-<pinref part="J3" gate="J1" pin="3"/>
-<wire x1="381" y1="-187.96" x2="378.46" y2="-187.96" width="0.1524" layer="91"/>
-</segment>
-</net>
-<net name="N$7" class="0">
-<segment>
-<pinref part="J3" gate="J1" pin="4"/>
-<wire x1="381" y1="-190.5" x2="378.46" y2="-190.5" width="0.1524" layer="91"/>
 </segment>
 </net>
@@
 </segment>
 </net>
+<net name="N$15" class="1">
+<segment>
+<pinref part="J1" gate="G$1" pin="24"/>
+<wire x1="243.84" y1="-73.66" x2="236.22" y2="-73.66" width="0.1524" layer="91"/>
+<pinref part="EPD_C12" gate="G$1" pin="2"/>
+</segment>
+</net>
+<net name="N$4" class="0">
+<segment>
+<pinref part="J2" gate="G$1" pin="B5"/>
+<wire x1="254" y1="25.4" x2="256.54" y2="25.4" width="0.1524" layer="91"/>
+<pinref part="R2-USB" gate="G$1" pin="1"/>
+</segment>
+</net>
